File: designs/arena_10_of_10_v1r1/column_buffer.kicad_sch (KiCad schematic)
At the start: 16 parts, among them U42 74LVC2G17, U43 74LVC2G17, U44 74LVC2G17, U45 74LVC2G17

Commit message: Tightened DRC rules, increased via sizes, and added switch
Added power switch SW1.

Assemble pin sockets for Teensy (J100/J101, 1x24 pin sockets; J102, 2x3 pin socket, 2mm pitch for ethernet).

Tightened board-setup DRC limits to match JLCPCB 6-layer minimums:

- min_hole_to_hole 0.25 -> 0.5 mm,
- min_text_thickness 0.08 -> 0.15 mm,
- min_via_annular_width 0.05 -> 0.075 mm.

Set stackup copper_finish from "None" to "ENIG".

Added PCB title block and automatic name / revision / date on silkscreen.

Refreshed footprints from library (0402/1210/SOT-23 crtyd now  uses fp_rect).

produced v1.1.2.
Other:
- company: (none) -> IORodeo for Reiser Lab @ Janelia | HHMI
- title: (none) -> G6 Teensy 10-10 Arena
Changed lines of the file:
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@@
 	(generator_version "9.0")
 	(paper "A4")
+	(title_block
+		(title "G6 Teensy 10-10 Arena")
+		(date "2026-04-22")
+		(rev "v1.1.2")
+		(company "IORodeo for Reiser Lab @ Janelia | HHMI")
+	)
 	(text "SN74LVC1G125DRLR\n296-18012-2-ND\n\n\nSN74HCS08BQAR\n296-SN74HCS08BQARTR-ND\n"
 		(exclude_from_sim no)
@@
 		)
 		(instances
-			(project ""
+			(project "arena_10_of_10_v1r1"
 				(path "/056666d2-2c8f-491c-bcad-db3c517779a8/3aea6610-f2a3-4b21-99b1-2866223bb12f/2d48c774-5bc7-44a4-9df6-3d6978bb1a97/9cbd2f9c-8fd6-45fc-a308-cb29b4b17e7c"
 					(reference "#PWR0414")
@@
 		)
 		(instances
-			(project ""
+			(project "arena_10_of_10_v1r1"
 				(path "/056666d2-2c8f-491c-bcad-db3c517779a8/3aea6610-f2a3-4b21-99b1-2866223bb12f/2d48c774-5bc7-44a4-9df6-3d6978bb1a97/9cbd2f9c-8fd6-45fc-a308-cb29b4b17e7c"
 					(reference "#PWR0424")
