File: arena_10-10/arena_top_10-10/panel_column.kicad_sch (KiCad schematic)
At the start: 4 parts, among them J5 Conn_01x05, J6 Conn_01x05, P1 NA

Commit message: produced v1.1.7
Parts:
- C42: MPN (none) -> HGC1210R5107M160NSVK
- J5, J6: MPN (none) -> 2.54-1*5P
Other:
- title: G6 Teensy 10-10 Arena -> G6 10-10 Arena Top
