File: arena_10-10/arena_top_10-10/panels.kicad_sch (KiCad schematic)
At the start: 0 parts

Commit message: produced v1.1.7
Other:
- title: G6 Teensy 10-10 Arena -> G6 10-10 Arena Top
Changed lines of the file:
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@@
 (kicad_sch
-	(version 20250114)
+	(version 20260306)
 	(generator "eeschema")
-	(generator_version "9.0")
+	(generator_version "10.0")
 	(paper "User" 279.4 304.8)
 	(title_block
-		(title "G6 Teensy 10-10 Arena")
-		(date "2026-04-28")
-		(rev "v1.1.7")
+		(title "G6 10-10 Arena Top")
+		(date "2026-05-26")
+		(rev "v1.1.0")
 		(company "IORodeo for Reiser Lab @ Janelia | HHMI")
 	)
@@
 		)
 		(fill
-			(color 255 255 194 1.0000)
+			(color 255 255 194 1)
 		)
 		(property "Sheetname" "Panel Column P8"
 			(at 175.26 95.8084 0)
+			(show_name no)
+			(do_not_autoplace no)
 			(effects
 				(font
@@
 		(property "Sheetfile" "panel_column.kicad_sch"
 			(at 175.26 119.9646 0)
+			(show_name no)
+			(do_not_autoplace no)
 			(effects
 				(font
@@
 		)
 		(fill
-			(color 255 255 194 1.0000)
+			(color 255 255 194 1)
 		)
 		(property "Sheetname" "Panel Column P10"
 			(at 175.26 161.8484 0)
+			(show_name no)
+			(do_not_autoplace no)
 			(effects
 				(font
@@
 		(property "Sheetfile" "panel_column.kicad_sch"
 			(at 175.26 186.0046 0)
+			(show_name no)
+			(do_not_autoplace no)
 			(effects
 				(font
@@
 		)
 		(fill
-			(color 255 255 194 1.0000)
+			(color 255 255 194 1)
 		)
 		(property "Sheetname" "Panel Column P1"
 			(at 106.68 31.0384 0)
+			(show_name no)
+			(do_not_autoplace no)
 			(effects
 				(font
@@
 		(property "Sheetfile" "panel_column.kicad_sch"
 			(at 106.68 55.1946 0)
+			(show_name no)
+			(do_not_autoplace no)
 			(effects
 				(font
@@
 		)
 		(fill
-			(color 255 255 194 1.0000)
+			(color 255 255 194 1)
 		)
 		(property "Sheetname" "Panel Column P3"
 			(at 106.68 95.8084 0)
+			(show_name no)
+			(do_not_autoplace no)
 			(effects
 				(font
@@
 		(property "Sheetfile" "panel_column.kicad_sch"
 			(at 106.68 119.9646 0)
+			(show_name no)
+			(do_not_autoplace no)
 			(effects
 				(font
@@
 		)
 		(fill
-			(color 255 255 194 1.0000)
+			(color 255 255 194 1)
 		)
 		(property "Sheetname" "Panel Column P9"
 			(at 175.26 128.8284 0)
+			(show_name no)
+			(do_not_autoplace no)
 			(effects
 				(font
@@
 		(property "Sheetfile" "panel_column.kicad_sch"
 			(at 175.26 152.9846 0)
+			(show_name no)
+			(do_not_autoplace no)
 			(effects
 				(font
@@
 		)
 		(fill
-			(color 255 255 194 1.0000)
+			(color 255 255 194 1)
 		)
 		(property "Sheetname" "Panel Column P6"
 			(at 175.26 31.0384 0)
+			(show_name no)
+			(do_not_autoplace no)
 			(effects
 				(font
@@
 		(property "Sheetfile" "panel_column.kicad_sch"
 			(at 175.26 55.1946 0)
+			(show_name no)
+			(do_not_autoplace no)
 			(effects
 				(font
@@
 		)
 		(fill
-			(color 255 255 194 1.0000)
+			(color 255 255 194 1)
 		)
 		(property "Sheetname" "Panel Column P2"
 			(at 106.68 62.7884 0)
+			(show_name no)
+			(do_not_autoplace no)
 			(effects
 				(font
@@
 		(property "Sheetfile" "panel_column.kicad_sch"
 			(at 106.68 86.9446 0)
+			(show_name no)
+			(do_not_autoplace no)
 			(effects
 				(font
@@
 		)
 		(fill
-			(color 255 255 194 1.0000)
+			(color 255 255 194 1)
 		)
 		(property "Sheetname" "Panel Column P5"
 			(at 106.68 161.8484 0)
+			(show_name no)
+			(do_not_autoplace no)
 			(effects
 				(font
@@
 		(property "Sheetfile" "panel_column.kicad_sch"
 			(at 106.68 186.0046 0)
+			(show_name no)
+			(do_not_autoplace no)
 			(effects
 				(font
@@
 		)
 		(fill
-			(color 255 255 194 1.0000)
+			(color 255 255 194 1)
 		)
 		(property "Sheetname" "Panel Column P4"
 			(at 106.68 128.8284 0)
+			(show_name no)
+			(do_not_autoplace no)
 			(effects
 				(font
@@
 		(property "Sheetfile" "panel_column.kicad_sch"
 			(at 106.68 152.9846 0)
+			(show_name no)
+			(do_not_autoplace no)
 			(effects
 				(font
@@
 		)
 		(fill
-			(color 255 255 194 1.0000)
+			(color 255 255 194 1)
 		)
 		(property "Sheetname" "Panel Column P7"
 			(at 175.26 62.7884 0)
+			(show_name no)
+			(do_not_autoplace no)
 			(effects
 				(font
@@
 		(property "Sheetfile" "panel_column.kicad_sch"
 			(at 175.26 86.9446 0)
-			(effects
-				(font
+			(show_name no)
+			(do_not_autoplace no)
+			(effects
+				(font
