File: arena_10-10/arena_top_10-10/power.kicad_sch (KiCad schematic)
At the start: 2 parts, among them J25 Barrel_Jack, SW1 SW_SPDT

Commit message: produced v1.1.7
Parts:
- J25: footprint arena_custom:DC-053D-20A -> arena_custom:BarrelJack_DC-053D-20A; MPN (none) -> DC-053D-20A
- SW1: MPN (none) -> HX SS12D10G6-WJ
Other:
- note removed: "Change DC Jack to PN DC-053D-20A Korean Hroparts Elec LCSC C707274"
- title: G6 Teensy 10-10 Arena -> G6 10-10 Arena Top
